Commit message: Fix collision box discrepancies between MoveIt and MuJoCo
- Fix object_sizes in simulation_server.py to match MuJoCo scene_breakfast.xml
  collision geom sizes exactly (cereal: [0.04,0.03] -> [0.035,0.023],
  banana y: 0.03 -> 0.02)
- Fix right_hand URDF collision from zero-size to proper cylinder
- Add missing right_gripper_base collision geometry
- Add collision detection instrumentation to run_task.py
  (snapshot_object_positions + detect_displacements)
- Add investigation summary doc in docs/collision_box_investigation.md

Co-Authored-By: Claude Opus 4.6 <noreply@anthropic.com>

File: src/assets/sawyer_with_electric_gripper.urdf (robot description, URDF)
Before this commit: robot sawyer, 33 links, 32 joints
Links:
- link right_gripper_base: geometry collision cylinder length=0.04 radius=0.035
- link right_hand: geometry collision cylinder length=0.05 radius=0.04
